Commit message: Update rplidar.urdf.xacro

File: sensors/rplidar.urdf.xacro (robot description, xacro)
@@ -1,5 +1,5 @@
 <?xml version="1.0"?>
 <robot name="rplidar" xmlns:xacro="http://wiki.ros.org/xacro">
-    <xacro:macro name="rplidar" params="name xyz rpy parent topic">
+    <xacro:macro name="rplidar" params="name xyz rpy parent min_a max_a topic:=scan">
         <link name="${name}">
             <visual>
