Commit message: add mesh for usb cam

File: sensors/usb_cam.urdf.xacro (robot description, xacro)
@@ -2,5 +2,24 @@
 <robot name="usb_cam" xmlns:xacro="http://wiki.ros.org/xacro">
     <xacro:macro name="usb_cam" params="name parent xyz rpy rate:=24">
-    <xacro:cube name="${name}" x="0.015" y="0.03" z="0.03" ori="-.007 0 0" rpy="0 0 0" rgb="Red" m="0.02" friction="${standard_friction}"/>
+    <link name="${name}">
+      <collision>
+          <origin xyz="0.0 0 0." rpy="0 0 0" />
+          <geometry>
+              <box size="0.025 0.05 0.05"/>
+          </geometry>
+      </collision>
+      <visual>
+          <origin xyz="0.0 0 0.0" rpy="0 ${pi/2} 0" />
+          <geometry>
+              <!-- <box size="0.025 0.05 0.05"/> -->
+              <mesh filename="file://$(find urdf_basic_shapes)/meshes/usb_cam.dae" scale="0.001 0.001 0.001" />
+          </geometry>
+      </visual>
+      <inertial>
+          <mass value="1e-5" />
+          <origin xyz="0.0 0 0.0" rpy="0 0 0" />
+          <inertia ixx="1e-6" ixy="0" ixz="0" iyy="1e-6" iyz="0" izz="1e-6" />
+      </inertial>
+  </link>
     <joint name="${name}_joint" type="fixed">
       <parent link="${parent}"/>
