Commit message: fix gps inertia

File: sensors/gps.urdf.xacro (robot description, xacro)
@@ -18,5 +18,5 @@
             <inertial>
                 <mass value="1e-5" />
-                <origin xyz="0 0 0" rpy="0 0 0" />
+                <origin xyz="0.01 0 0.061" rpy="${pi/2} 0 0" />
                 <inertia ixx="1e-6" ixy="0" ixz="0" iyy="1e-6" iyz="0" izz="1e-6" />
             </inertial>
