Commit message: add param for imu freq

File: sensors/imu.urdf.xacro (robot description, xacro)
@@ -1,5 +1,5 @@
 <?xml version="1.0"?>
 <robot name="imu" xmlns:xacro="http://wiki.ros.org/xacro">
-    <xacro:macro name="imu" params="name parent xyz rpy">
+    <xacro:macro name="imu" params="name parent xyz rpy hz:=100">
         <link name="${name}" />
         <joint name="${name}_joint" type="fixed">
@@ -14,5 +14,5 @@
             <sensor name="${name}" type="imu">
                 <always_on>true</always_on>
-                <update_rate>200</update_rate>
+                <update_rate>${hz}</update_rate>
                 <visualize>true</visualize>
                 <topic>${name}</topic>
